Commit message: edit

File: models/diff_drive_robot/urdf/diff_drive_robot.xacro (robot description, xacro)
@@ -1,6 +1,6 @@
 <?xml version='1.0'?>
 <robot name="robot" xmlns:xacro="http://www.ros.org/wiki/xacro">
-  <xacro:include filename="$(find roscourse_2023_project_scene)/models/diff_drive_robot/urdf/diff_drive_robot.gazebo" />
-  <xacro:include filename="$(find roscourse_2023_project_scene)/models/diff_drive_robot/urdf/materials.xacro" />
+  <xacro:include filename="$(find project)/models/diff_drive_robot/urdf/diff_drive_robot.gazebo" />
+  <xacro:include filename="$(find project)/models/diff_drive_robot/urdf/materials.xacro" />
   <link name='base'>
     <pose>0 0 0.0 0 0 0</pose>
@@ -121,13 +121,58 @@
     </inertial>
   </link>
+  <!-- <link name='camera'>
+    <visual name='camera_visual'>
+      <origin xyz="0 0 0" rpy=" 0 0 0"/>
+      <geometry>
+        <box size=".05 .05 .05"/>
+      </geometry>
+      <material name="white"/>
+    </visual>
+  </link>
   <link name='camera2'>
-    <visual name='camera_visual'>
-      <origin xyz="0 0 0" rpy=" 0 0 0"/>
-      <geometry>
-        <box size=".05 .05 .05"/>
-      </geometry>
-      <material name="white"/>
-    </visual>
-  </link>
+    <visual name='camera_visual2'>
+      <origin xyz="0 0 0" rpy=" 0 0 0"/>
+      <geometry>
+        <box size=".05 .05 .05"/>
+      </geometry>
+      <material name="white"/>
+    </visual>
+  </link> -->
+  <!-- <link name='depth_camera'>
+    <visual name='depth_camera_visual'>
+      <origin xyz="0 0 0" rpy=" 0 0 0"/>
+      <geometry>
+        <box size=".05 .05 .05"/>
+      </geometry>
+      <material name="white"/>
+    </visual>
+  </link>
+  <link name='depth_camera2'>
+    <visual name='depth_camera_visual2'>
+      <origin xyz="0 0 0" rpy=" 0 0 0"/>
+      <geometry>
+        <box size=".05 .05 .05"/>
+      </geometry>
+      <material name="white"/>
+    </visual>
+  </link> -->
+  <link name='lidar'>
+    <visual name='lidar_visual'>
+      <origin xyz="0 0 0" rpy=" 0 0 0"/>
+      <geometry>
+        <box size=".05 .05 .05"/>
+      </geometry>
+      <material name="white"/>
+    </visual>
+  </link>
+  <!-- <link name='lidar2'>
+    <visual name='lidar2_visual'>
+      <origin xyz="0 0 0" rpy=" 0 0 0"/>
+      <geometry>
+        <box size=".05 .05 .05"/>
+      </geometry>
+      <material name="white"/>
+    </visual>
+  </link> -->
   <joint type="continuous" name="left_wheel_hinge">
     <origin xyz="0.05 0.226 -0.05" rpy="0 0 0"/>
@@ -138,4 +183,14 @@
     <joint_properties damping="0.0" friction="0.0"/>
   </joint>
+  <transmission name="left_wheel_trans">
+      <type>transmission_interface/SimpleTransmission</type>
+      <joint name="left_wheel_hinge">
+         <hardwareInterface>EffortJointInterface</hardwareInterface>
+      </joint>
+      <actuator name="left_wheel_motor">
+         <hardwareInterface>EffortJointInterface</hardwareInterface>
+         <mechanicalReduction>1</mechanicalReduction>
+      </actuator>
+  </transmission>
   <joint type="continuous" name="right_wheel_hinge">
     <origin xyz="0.05 -0.226 -0.05" rpy="0 0 0"/>
@@ -146,8 +201,44 @@
     <joint_properties damping="0.0" friction="0.0"/>
   </joint>
-  <joint type="fixed" name="camera_joint">
-    <origin xyz="0.3 0 0" rpy="0 0 0"/>
+  <transmission name="right_wheel_trans">
+      <type>transmission_interface/SimpleTransmission</type>
+      <joint name="right_wheel_hinge">
+         <hardwareInterface>EffortJointInterface</hardwareInterface>
+      </joint>
+      <actuator name="right_wheel_motor">
+         <hardwareInterface>EffortJointInterface</hardwareInterface>
+         <mechanicalReduction>1</mechanicalReduction>
+      </actuator>
+  </transmission>
+  <!-- <joint type="fixed" name="camera_joint">
+    <origin xyz="0.3 0.1 0" rpy="0 0 0"/>
+    <child link="camera"/>
+    <parent link="base"/>
+  </joint>
+  <joint type="fixed" name="depth_camera_joint">
+    <origin xyz="0.3 -0.1 0" rpy="0 0 0"/>
+    <child link="depth_camera"/>
+    <parent link="base"/>
+  </joint>
+  <joint type="fixed" name="camera_joint2">
+    <origin xyz="-0.3 0.1 0" rpy="0 0 ${pi}"/>
     <child link="camera2"/>
     <parent link="base"/>
   </joint>
+  <joint type="fixed" name="depth_camera_joint2">
+    <origin xyz="-0.3 -0.1 0" rpy="0 0 ${pi}"/>
+    <child link="depth_camera2"/>
+    <parent link="base"/>
+  </joint> -->
+  <joint type="fixed" name="lidar_joint">
+    <origin xyz="0.3 0.1 0" rpy="0 0 -${pi/2}"/>
+    <child link="lidar"/>
+    <parent link="base"/>
+  </joint>
+<!--
+  <joint type="fixed" name="lidar2_joint">
+    <origin xyz="0 -0.15 0.125" rpy="0 0 ${pi}"/>
+    <child link="lidar2"/>
+    <parent link="base"/>
+  </joint> -->
 </robot>

Commit message: lidar fix

File: models/diff_drive_robot/urdf/diff_drive_robot.xacro (robot description, xacro)
@@ -232,5 +232,5 @@
   </joint> -->
   <joint type="fixed" name="lidar_joint">
-    <origin xyz="0.3 0.1 0" rpy="0 0 -${pi/2}"/>
+    <origin xyz="0.3 0.0 0" rpy="0 0 -${pi/2}"/>
     <child link="lidar"/>
     <parent link="base"/>

Commit message: fix inertial

File: models/diff_drive_robot/urdf/diff_drive_robot.xacro (robot description, xacro)
@@ -3,15 +3,10 @@
   <xacro:include filename="$(find project)/models/diff_drive_robot/urdf/diff_drive_robot.gazebo" />
   <xacro:include filename="$(find project)/models/diff_drive_robot/urdf/materials.xacro" />
+  <xacro:include filename="$(find project)/models/diff_drive_robot/urdf/inertial.usdf.xacro" />
   <link name='base'>
     <pose>0 0 0.0 0 0 0</pose>
-    <inertial>
-      <mass value="20.0"/>
+    <xacro:inertial_box mass="10.0" x="0.6" y="0.4" z="0.2">
       <origin xyz="0.0 0 0.1" rpy=" 0 0 0"/>
-      <inertia
-          ixx="0.5" ixy="0" ixz="0"
-          iyy="1.0" iyz="0"
-          izz="0.1"
-      />
-    </inertial>
+    </xacro:inertial_box>
     <collision name='collision'>
       <geometry>
@@ -87,13 +82,7 @@
       <material name="green"/>
     </visual>
-    <inertial>
-      <origin xyz="0 0 0" rpy="0 1.5707 1.5707"/>
-      <mass value="5"/>
-      <cylinder_inertia m="5" r="0.1" h="0.05"/>
-      <inertia
-        ixx="1.0" ixy="0.0" ixz="0.0"
-        iyy="1.0" iyz="0.0"
-        izz="1.0"/>
-    </inertial>
+    <xacro:inertial_cylinder mass="5.0" length="0.05" radius="0.1">
+      <origin xyz="0 0 0" rpy="0 1.5707 1.5707"/>
+    </xacro:inertial_cylinder>
   </link>
   <link name="right_wheel">
@@ -111,13 +100,7 @@
       <material name="green"/>
     </visual>
-    <inertial>
-      <origin xyz="0 0 0" rpy="0 1.5707 1.5707"/>
-      <mass value="5"/>
-      <cylinder_inertia m="5" r="0.1" h="0.05"/>
-      <inertia
-        ixx="1.0" ixy="0.0" ixz="0.0"
-        iyy="1.0" iyz="0.0"
-        izz="1.0"/>
-    </inertial>
+    <xacro:inertial_cylinder mass="5.0" length="0.05" radius="0.1">
+      <origin xyz="0 0 0" rpy="0 1.5707 1.5707"/>
+    </xacro:inertial_cylinder>
   </link>
   <!-- <link name='camera'>
